Commit message: update: GO2 urdf and usd

File: source/GO2/assets/urdf/go2/urdf/go2.urdf (robot description, URDF)
Before this commit: robot go2_description, 29 links, 28 joints
Links:
- link FL_calf: geometry collision cylinder length=0.05 radius=0.01; visual mesh filename=../dae/calf.dae
- link FL_thigh: geometry collision box size=0.16 0.0245 0.034; visual mesh filename=../dae/thigh.dae
- link FR_calf: geometry collision cylinder length=0.05 radius=0.01; visual mesh filename=../dae/calf_mirror.dae
- link FR_thigh: geometry collision box size=0.16 0.0245 0.034; visual mesh filename=../dae/thigh_mirror.dae
- link RL_calf: geometry collision cylinder length=0.05 radius=0.01; visual mesh filename=../dae/calf.dae
- link RL_thigh: geometry collision box size=0.16 0.0245 0.034; visual mesh filename=../dae/thigh.dae
- link RR_calf: geometry collision cylinder length=0.05 radius=0.01; visual mesh filename=../dae/calf_mirror.dae
- link RR_thigh: geometry collision box size=0.16 0.0245 0.034; visual mesh filename=../dae/thigh_mirror.dae
